File: pcb/01_POWER.kicad_sch (KiCad schematic)
At the start: 15 parts, among them M1 LM2596HVS 5V, U11 AP2112K-3.3

Commit message: pcb: S12 relay-expansion integration + R1/R2 e-stop fixes (schematic + board)
- 09_EMERGENCY: R1 fix (active-LOW drive: R72 high-side from +3V3, OPT1 cathode
  -> RELAY_CTRL, R78 10k pull-up fail-safe) + R2 fix (inverting sense: Q21
  BSS138 + R77 100k divider + R76 revalued 10k pull-up, C75 filter; HIGH=trip
  matches GPIO14 INPUT_PULLUP contract); truth table/docs updated
- NEW 12_RELAY_EXP: F4 1.1A + FB2 -> +5V_RELAY_EXP rail, J_RELAY_EXP 2x03,
  BSS138 I2C shifters Q22/Q23 + R79/R84 4k7, TVS D24/D25 DNP, INT divider
  R82/R83 (PCF8574 module external, 0x20, active-LOW)
- root sch: sheet 12 entry (page 13); plts-custom: +5V_RELAY_EXP symbol
- pro: PWR netclass pattern for +5V_RELAY_EXP
- 01_POWER: C52 22uF->47uF 25V X5R (relay coil dip headroom)
- board: +7 nets, +14 footprints, pad re-netting, placement to 0 structural
  DRC; repaired broken hand-drawn courtyards (M1/U1/K1/J_I2C_EXP) to true
  geometry; U1 antenna keepout respected

ERC: 0 violations (13 sheets). DRC: 0 structural (courtyard/short/keepout/
clearance clean; silk/via/thermal/isolated = post-routing cleanup).
Parts:
- C52: value 22uF 25V X7R -> 47uF 25V X5R
Changed lines of the file:
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@@
 			(effects (font (size 1.27 1.27)) (justify right))
 		)
-		(property "Value" "22uF 25V X7R"
+		(property "Value" "47uF 25V X5R"
 			(at 241.3 116.84 0)
 			(effects (font (size 1.27 1.27)) (justify left))
